File: Battery-Management.kicad_sch (KiCad schematic)
At the start: 13 parts, among them U3 MCP73831-2-MC, U4 TC2185-3.3VxCTTR

Commit message: Added USB C and CAN interfaces to schematic
Connections:
- net +3.3V: no longer C5.1, U4.5 (VOUT)
- new net: C5.1, U4.5 (VOUT)
Changed lines of the file:
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@@
-	)
-	(junction
-		(at 167.64 134.62)
-		(diameter 0)
-		(color 0 0 0 0)
 	)
 	(junction
@@
 	(wire
 		(pts
-			(xy 167.64 132.08) (xy 167.64 134.62)
-		)
-		(stroke
-			(width 0)
-			(type default)
-		)
-	)
-	(wire
-		(pts
 			(xy 163.83 109.22) (xy 176.53 109.22)
 		)
@@
 			(width 0)
 			(type default)
+		)
+	)
+	(text_box "ONLY D1 on: Charging\nONLY D2 on: Done charging\nD1 & D2 on: BMS in shutdown mode\nD1 & D2 off: No power from USB"
+		(exclude_from_sim no)
+		(at 223.52 92.71 0)
+		(size 40.64 10.16)
+		(stroke
+			(width 0)
+			(type default)
+		)
+		(fill
+			(type none)
+		)
+		(effects
+			(font
+				(size 1.27 1.27)
+			)
+			(justify left top)
 		)
 	)
@@
 	(symbol
 		(lib_id "power:+3.3V")
-		(at 167.64 132.08 0)
+		(at 185.42 129.54 0)
 		(unit 1)
 		(exclude_from_sim no)
@@
 		(fields_autoplaced yes)
 		(property "Reference" "#PWR018"
-			(at 167.64 135.89 0)
+			(at 185.42 133.35 0)
 			(effects
 				(font
@@
 		)
 		(property "Value" "+3.3V"
-			(at 167.64 127 0)
+			(at 185.42 124.46 0)
 			(effects
 				(font
@@
 		)
 		(property "Footprint" ""
-			(at 167.64 132.08 0)
+			(at 185.42 129.54 0)
 			(effects
 				(font
@@
 		)
 		(property "Datasheet" ""
-			(at 167.64 132.08 0)
+			(at 185.42 129.54 0)
 			(effects
 				(font
@@
 		)
 		(property "Description" "Power symbol creates a global label with name \"+3.3V\""
-			(at 167.64 132.08 0)
-			(effects
-				(font
+			(at 185.42 129.54 0)
+			(effects
+				(font

Commit message: New, simpler CAN interface that supports FD CAN
Connections:
- net +3.3V: now also C5.1, U4.5 (VOUT)
Changed lines of the file:
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@@
+	)
+	(junction
+		(at 167.64 134.62)
+		(diameter 0)
+		(color 0 0 0 0)
 	)
 	(junction
@@
 		(pts
 			(xy 149.86 137.16) (xy 153.67 137.16)
+		)
+		(stroke
+			(width 0)
+			(type default)
+		)
+	)
+	(wire
+		(pts
+			(xy 167.64 130.81) (xy 167.64 134.62)
 		)
 		(stroke
@@
 	(symbol
 		(lib_id "power:+3.3V")
-		(at 185.42 129.54 0)
+		(at 167.64 130.81 0)
 		(unit 1)
 		(exclude_from_sim no)
@@
 		(fields_autoplaced yes)
 		(property "Reference" "#PWR018"
-			(at 185.42 133.35 0)
+			(at 167.64 134.62 0)
 			(effects
 				(font
@@
 		)
 		(property "Value" "+3.3V"
-			(at 185.42 124.46 0)
+			(at 167.64 125.73 0)
 			(effects
 				(font
@@
 		)
 		(property "Footprint" ""
-			(at 185.42 129.54 0)
+			(at 167.64 130.81 0)
 			(effects
 				(font
@@
 		)
 		(property "Datasheet" ""
-			(at 185.42 129.54 0)
+			(at 167.64 130.81 0)
 			(effects
 				(font
@@
 		)
 		(property "Description" "Power symbol creates a global label with name \"+3.3V\""
-			(at 185.42 129.54 0)
-			(effects
-				(font
+			(at 167.64 130.81 0)
+			(effects
+				(font

Commit message: Routed USB interface from port to MCU and CAN interface from connector to transceiver
Parts:
- removed BT1: BH-18650-PC, Battery:BatteryHolder_MPD_BH-18650-PC2, symbol BH-18650-PC:BH-18650-PC
- added BT1: Battery_Cell, Battery:BatteryHolder_MPD_BH-18650-PC2, symbol Device:Battery_Cell
Connections:
- net GNDD: now also BT1.2 (-)
- net V_BAT: now also BT1.1 (+)
Changed lines of the file:
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@@
 	(paper "A4")
+	(junction
+		(at 167.64 134.62)
+		(diameter 0)
+		(color 0 0 0 0)
+	)
 	(junction
 		(at 176.53 96.52)
@@
 	)
 	(junction
-		(at 167.64 134.62)
-		(diameter 0)
-		(color 0 0 0 0)
-	)
-	(junction
 		(at 163.83 96.52)
 		(diameter 0)
@@
 	(wire
 		(pts
+			(xy 176.53 106.68) (xy 176.53 109.22)
+		)
+		(stroke
+			(width 0)
+			(type default)
+		)
+	)
+	(wire
+		(pts
 			(xy 176.53 109.22) (xy 176.53 111.76)
 		)
@@
 	(wire
 		(pts
+			(xy 176.53 96.52) (xy 176.53 99.06)
+		)
+		(stroke
+			(width 0)
+			(type default)
+		)
+	)
+	(wire
+		(pts
 			(xy 121.92 146.05) (xy 121.92 147.32)
 		)
@@
 	(wire
 		(pts
-			(xy 185.42 96.52) (xy 176.53 96.52)
-		)
-		(stroke
-			(width 0)
-			(type default)
-		)
-	)
-	(wire
-		(pts
 			(xy 149.86 134.62) (xy 167.64 134.62)
 		)
@@
 		(pts
 			(xy 149.86 82.55) (xy 140.97 82.55)
+		)
+		(stroke
+			(width 0)
+			(type default)
+		)
+	)
+	(wire
+		(pts
+			(xy 176.53 96.52) (xy 185.42 96.52)
 		)
 		(stroke
@@
 	)
 	(symbol
-		(lib_id "BH-18650-PC:BH-18650-PC")
-		(at 176.53 104.14 270)
-		(unit 1)
-		(exclude_from_sim no)
-		(in_bom yes)
-		(on_board yes)
-		(dnp no)
-		(fields_autoplaced yes)
-		(property "Reference" "BT1"
-			(at 180.34 100.3299 90)
-			(effects
-				(font
-					(size 1.27 1.27)
-				)
-				(justify left)
-			)
-		)
-		(property "Value" "BH-18650-PC"
-			(at 180.34 102.8699 90)
-			(effects
-				(font
-					(size 1.27 1.27)
-				)
-				(justify left)
-			)
-		)
-		(property "Footprint" "Battery:BatteryHolder_MPD_BH-18650-PC2"
-			(at 176.53 104.14 0)
-			(effects
-				(font
-					(size 1.27 1.27)
-				)
-				(justify bottom)
-				(hide yes)
-			)
-		)
-		(property "Datasheet" ""
-			(at 176.53 104.14 0)
-			(effects
-				(font
-					(size 1.27 1.27)
-				)
-				(hide yes)
-			)
-		)
-		(property "Description" ""
-			(at 176.53 104.14 0)
-			(effects
-				(font
-					(size 1.27 1.27)
-				)
-				(hide yes)
-			)
-		)
-		(property "PARTREV" "05/17/19"
-			(at 176.53 104.14 0)
-			(effects
-				(font
-					(size 1.27 1.27)
-				)
-				(justify bottom)
-				(hide yes)
-			)
-		)
-		(property "STANDARD" "Manufacturer Recommendation"
-			(at 176.53 104.14 0)
-			(effects
-				(font
-					(size 1.27 1.27)
-				)
-				(justify bottom)
-				(hide yes)
-			)
-		)
-		(property "MAXIMUM_PACKAGE_HEIGHT" "21.31mm"
-			(at 176.53 104.14 0)
-			(effects
-				(font
-					(size 1.27 1.27)
-				)
-				(justify bottom)
-				(hide yes)
-			)
-		)
-		(property "MANUFACTURER" "MPD"
-			(at 176.53 104.14 0)
-			(effects
-				(font
-					(size 1.27 1.27)
-				)
-				(justify bottom)
-				(hide yes)
-			)
-		)
-		(pin "P"
-		)
-		(pin "N"
-		)
-		(instances
-			(project ""
-				(path "/c41b490b-5ab6-4438-aea0-388670bb08f4/b5b03a48-538a-4431-9fe0-db318c963946"
-					(reference "BT1")
-					(unit 1)
-				)
-			)
-		)
-	)
-	(symbol
 		(lib_id "Device:C")
 		(at 121.92 142.24 0)
@@
 					(unit 1)
 				)
+			)
+		)
+	)
+	(symbol
+		(lib_id "Device:Battery_Cell")
+		(at 176.53 104.14 0)
+		(unit 1)
+		(exclude_from_sim no)
+		(in_bom yes)
+		(on_board yes)
+		(dnp no)
+		(fields_autoplaced yes)
+		(property "Reference" "BT1"
+			(at 180.34 101.0284 0)
+			(effects
+				(font
+					(size 1.27 1.27)
+				)
+				(justify left)
+			)
+		)
+		(property "Value" "Battery_Cell"
+			(at 180.34 103.5684 0)
+			(effects
+				(font
+					(size 1.27 1.27)
+				)
+				(justify left)
+			)
+		)
+		(property "Footprint" "Battery:BatteryHolder_MPD_BH-18650-PC2"
+			(at 176.53 102.616 90)
+			(effects
+				(font
+					(size 1.27 1.27)
+				)
+				(hide yes)
+			)
+		)
+		(property "Datasheet" "~"
+			(at 176.53 102.616 90)
+			(effects
+				(font
+					(size 1.27 1.27)
+				)
+				(hide yes)
+			)
+		)
+		(property "Description" "Single-cell battery"
+			(at 176.53 104.14 0)
+			(effects
+				(font
+					(size 1.27 1.27)
+				)
+				(hide yes)
+			)
+		)
+		(pin "2"
+		)
+		(pin "1"
+		)
+		(instances
+			(project ""
+				(path "/c41b490b-5ab6-4438-aea0-388670bb08f4/b5b03a48-538a-4431-9fe0-db318c963946"
+					(reference "BT1")
+					(unit 1)
+				)
