File: USB-C-Interface.kicad_sch (KiCad schematic)
At the start: 0 parts

Commit message: Added USB C and CAN interfaces to schematic
Parts:
- added CR1: ESDA7P60-1U1M, ZDO_1610_STM, symbol 2024-07-15_00-58-56:ESDA7P60-1U1M
- added J3: USB_C_Receptacle_USB2.0_16P, Connector_USB:USB_C_Receptacle_GCT_USB4105-xx-A_16P_TopMnt_Horizontal, symbol Connector:USB_C_Receptacle_USB2.0_16P
- added R2, R5: 5.1k, Resistor_SMD:R_0603_1608Metric_Pad0.98x0.95mm_HandSolder, symbol Device:R_US
- added TP4: TestPoint, symbol Connector:TestPoint
- added U5: USBLC6-2SC6, Package_TO_SOT_SMD:SOT-23-6, symbol Power_Protection:USBLC6-2SC6
Connections:
- new net: J3.A7 (D-), J3.B7 (D-), U5.1 (I/O1)
- new net: J3.A6 (D+), J3.B6 (D+), U5.3 (I/O2)
- new net: J3.A5 (CC1), R2.1
- new net: J3.B5 (CC2), R5.1
- new net GNDD: CR1.2, J3.A1 (GND), J3.A12 (GND), J3.B1 (GND), J3.B12 (GND), J3.S1 (SHIELD), R2.2, R5.2, U5.2 (GND)
- new net USB_D_N: U5.6 (I/O1)
- new net USB_D_P: U5.4 (I/O2)
- new net V_USB: CR1.1, J3.A4 (VBUS), J3.A9 (VBUS), J3.B4 (VBUS), J3.B9 (VBUS), TP4.1
- no-connect marks 0 -> 3

Commit message: Routed USB interface from port to MCU and CAN interface from connector to transceiver
Parts:
- TP4: footprint (none) -> TestPoint:TestPoint_Loop_D2.60mm_Drill1.6mm_Beaded
