File: pcb/sensors.kicad_sch (KiCad schematic)
At the start: 5 parts, among them U1 MS5607-02BA, U7 ADXL375BCCZ

Commit message: Routed reset monitor, all test points, 128 MBit flash, sensors, analog-digital jumper switches
Connections:
- net accel_cs is gone; now on net GNDD: U7.7 (*CS)
- net pres_cs is gone; now on net GNDD: U1.4 (CSB), U1.5 (CSB)
- net +3.3V: now also C19.1, C20.1, U7.1 (VDD_I/O), U7.6 (VS)
Changed lines of the file:
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@@
-	(wire
-		(pts
-			(xy 62.23 92.71) (xy 62.23 95.25)
-		)
-		(stroke
-			(width 0)
-			(type default)
-		)
-	)
 	(wire
 		(pts
@@
 	(wire
 		(pts
+			(xy 142.24 87.63) (xy 142.24 88.9)
+		)
+		(stroke
+			(width 0)
+			(type default)
+		)
+	)
+	(wire
+		(pts
 			(xy 78.74 81.28) (xy 78.74 83.82)
 		)
@@
 	(wire
 		(pts
-			(xy 60.96 92.71) (xy 62.23 92.71)
+			(xy 53.34 95.25) (xy 68.58 95.25)
 		)
 		(stroke
@@
 		(pts
 			(xy 152.4 88.9) (xy 142.24 88.9)
-		)
-		(stroke
-			(width 0)
-			(type default)
-		)
-	)
-	(wire
-		(pts
-			(xy 62.23 95.25) (xy 68.58 95.25)
 		)
 		(stroke
@@
 		)
 	)
-	(hierarchical_label "pres_cs"
+	(hierarchical_label "accel_mosi"
 		(shape input)
-		(at 53.34 105.41 180)
+		(at 152.4 104.14 180)
 		(fields_autoplaced yes)
 		(effects
@@
 		)
 	)
-	(hierarchical_label "accel_cs"
+	(hierarchical_label "pres_mosi"
 		(shape input)
-		(at 152.4 114.3 180)
+		(at 53.34 100.33 180)
 		(fields_autoplaced yes)
 		(effects
@@
 		)
 	)
-	(hierarchical_label "accel_mosi"
-		(shape input)
-		(at 152.4 104.14 180)
+	(hierarchical_label "accel_miso"
+		(shape output)
+		(at 152.4 109.22 180)
 		(fields_autoplaced yes)
 		(effects
@@
 		)
 	)
-	(hierarchical_label "pres_mosi"
-		(shape input)
-		(at 53.34 100.33 180)
+	(hierarchical_label "accel_int2"
+		(shape output)
+		(at 228.6 91.44 0)
 		(fields_autoplaced yes)
 		(effects
@@
 				(size 1.27 1.27)
 			)
-			(justify right)
-		)
-	)
-	(hierarchical_label "accel_miso"
+			(justify left)
+		)
+	)
+	(hierarchical_label "pres_miso"
 		(shape output)
-		(at 152.4 109.22 180)
+		(at 53.34 97.79 180)
 		(fields_autoplaced yes)
 		(effects
@@
 		)
 	)
-	(hierarchical_label "accel_int2"
-		(shape output)
-		(at 228.6 91.44 0)
+	(hierarchical_label "accel_sclk"
+		(shape bidirectional)
+		(at 152.4 99.06 180)
 		(fields_autoplaced yes)
 		(effects
@@
 				(size 1.27 1.27)
 			)
-			(justify left)
-		)
-	)
-	(hierarchical_label "pres_miso"
-		(shape output)
-		(at 53.34 97.79 180)
-		(fields_autoplaced yes)
-		(effects
-			(font
-				(size 1.27 1.27)
-			)
 			(justify right)
 		)
 	)
-	(hierarchical_label "accel_sclk"
-		(shape bidirectional)
-		(at 152.4 99.06 180)
-		(fields_autoplaced yes)
-		(effects
-			(font
-				(size 1.27 1.27)
-			)
-			(justify right)
-		)
-	)
 	(symbol
 		(lib_id "power:GNDD")
-		(at 60.96 92.71 270)
+		(at 53.34 95.25 270)
 		(unit 1)
 		(exclude_from_sim no)
@@
 		(fields_autoplaced yes)
 		(property "Reference" "#PWR033"
-			(at 54.61 92.71 0)
+			(at 46.99 95.25 0)
 			(effects
 				(font
@@
 		)
 		(property "Value" "GNDD"
-			(at 57.15 92.7099 90)
+			(at 49.53 95.2499 90)
 			(effects
 				(font
@@
 		)
 		(property "Footprint" ""
-			(at 60.96 92.71 0)
+			(at 53.34 95.25 0)
 			(effects
 				(font
@@
 		)
 		(property "Datasheet" ""
-			(at 60.96 92.71 0)
+			(at 53.34 95.25 0)
 			(effects
 				(font
@@
 		)
 		(property "Description" "Power symbol creates a global label with name \"GNDD\" , digital ground"
-			(at 60.96 92.71 0)
+			(at 53.34 95.25 0)
 			(effects
 				(font
@@
 	)
 	(symbol
+		(lib_id "power:GNDD")
+		(at 152.4 114.3 270)
+		(unit 1)
+		(exclude_from_sim no)
+		(in_bom yes)
+		(on_board yes)
+		(dnp no)
+		(fields_autoplaced yes)
+		(property "Reference" "#PWR043"
+			(at 146.05 114.3 0)
+			(effects
+				(font
+					(size 1.27 1.27)
+				)
+				(hide yes)
+			)
+		)
+		(property "Value" "GNDD"
+			(at 148.59 114.2999 90)
+			(effects
+				(font
+					(size 1.27 1.27)
+				)
+				(justify right)
+			)
+		)
+		(property "Footprint" ""
+			(at 152.4 114.3 0)
+			(effects
+				(font
+					(size 1.27 1.27)
+				)
+				(hide yes)
+			)
+		)
+		(property "Datasheet" ""
+			(at 152.4 114.3 0)
+			(effects
+				(font
+					(size 1.27 1.27)
+				)
+				(hide yes)
+			)
+		)
+		(property "Description" "Power symbol creates a global label with name \"GNDD\" , digital ground"
+			(at 152.4 114.3 0)
+			(effects
+				(font
+					(size 1.27 1.27)
+				)
+				(hide yes)
+			)
+		)
+		(pin "1"
+		)
+		(instances
+			(project ""
+				(path "/c41b490b-5ab6-4438-aea0-388670bb08f4/3e9e0b47-da2c-4332-b911-05c7ab3ede69"
+					(reference "#PWR043")
+					(unit 1)
+				)
+			)
+		)
+	)
+	(symbol
 		(lib_id "power:+3.3V")
 		(at 78.74 81.28 0)
@@
 	(symbol
 		(lib_id "power:GNDD")
+		(at 53.34 105.41 270)
+		(unit 1)
+		(exclude_from_sim no)
+		(in_bom yes)
+		(on_board yes)
+		(dnp no)
+		(fields_autoplaced yes)
+		(property "Reference" "#PWR044"
+			(at 46.99 105.41 0)
+			(effects
+				(font
+					(size 1.27 1.27)
+				)
+				(hide yes)
+			)
+		)
+		(property "Value" "GNDD"
+			(at 49.53 105.4099 90)
+			(effects
+				(font
+					(size 1.27 1.27)
+				)
+				(justify right)
+			)
+		)
+		(property "Footprint" ""
+			(at 53.34 105.41 0)
+			(effects
+				(font
+					(size 1.27 1.27)
+				)
+				(hide yes)
+			)
+		)
+		(property "Datasheet" ""
+			(at 53.34 105.41 0)
+			(effects
+				(font
+					(size 1.27 1.27)
+				)
+				(hide yes)
+			)
+		)
+		(property "Description" "Power symbol creates a global label with name \"GNDD\" , digital ground"
+			(at 53.34 105.41 0)
+			(effects
+				(font
+					(size 1.27 1.27)
+				)
+				(hide yes)
+			)
+		)
+		(pin "1"
+		)
+		(instances
+			(project ""
+				(path "/c41b490b-5ab6-4438-aea0-388670bb08f4/3e9e0b47-da2c-4332-b911-05c7ab3ede69"
+					(reference "#PWR044")
+					(unit 1)
+				)
+			)
+		)
+	)
+	(symbol
+		(lib_id "power:GNDD")
 		(at 90.17 91.44 0)
 		(unit 1)
@@
 					(unit 1)
 				)
+			)
+		)
+	)
+	(symbol
+		(lib_id "power:+3.3V")
+		(at 142.24 87.63 0)
+		(unit 1)
+		(exclude_from_sim no)
+		(in_bom yes)
+		(on_board yes)
+		(dnp no)
+		(fields_autoplaced yes)
+		(property "Reference" "#PWR047"
+			(at 142.24 91.44 0)
+			(effects
+				(font
+					(size 1.27 1.27)
+				)
+				(hide yes)
+			)
+		)
+		(property "Value" "+3.3V"
+			(at 142.24 82.55 0)
+			(effects
+				(font
+					(size 1.27 1.27)
+				)
+			)
+		)
+		(property "Footprint" ""
+			(at 142.24 87.63 0)
+			(effects
+				(font
+					(size 1.27 1.27)
+				)
+				(hide yes)
+			)
+		)
+		(property "Datasheet" ""
+			(at 142.24 87.63 0)
+			(effects
+				(font
+					(size 1.27 1.27)
+				)
+				(hide yes)
+			)
+		)
+		(property "Description" "Power symbol creates a global label with name \"+3.3V\""
+			(at 142.24 87.63 0)
+			(effects
+				(font
+					(size 1.27 1.27)
+				)
+				(hide yes)
+			)
+		)
+		(pin "1"
+		)
+		(instances
+			(project ""
+				(path "/c41b490b-5ab6-4438-aea0-388670bb08f4/3e9e0b47-da2c-4332-b911-05c7ab3ede69"
+					(reference "#PWR047")
+					(unit 1)
+				)
