File: Common/USB-C-Interface.kicad_sch (KiCad schematic)
At the start: 6 parts

Commit message: Added footprints for GPS module, new edge cuts for main module
Parts:
- USB_CR1: footprint ESDA7P60:ZDO_1610_STM -> ESDA7P60_1U1M:ZDO_1610_STM
Changed lines of the file:
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@@
 		(instances
+			(project "Main-Module"
+				(path "/acc63f22-7eb8-450a-9af4-da5f4b8157d9/066db7ca-fd8b-46d1-a06b-412eb11482f3"
+					(reference "USB_U1")
+					(unit 1)
+				)
+			)
 			(project "Main-Module"
 				(path "/c41b490b-5ab6-4438-aea0-388670bb08f4/b23d16a1-3c5b-4321-8b30-5d6992e2f62d"
@@
 		(instances
 			(project "Main-Module"
+				(path "/acc63f22-7eb8-450a-9af4-da5f4b8157d9/066db7ca-fd8b-46d1-a06b-412eb11482f3"
+					(reference "USB_J1")
+					(unit 1)
+				)
+			)
+			(project "Main-Module"
 				(path "/c41b490b-5ab6-4438-aea0-388670bb08f4/b23d16a1-3c5b-4321-8b30-5d6992e2f62d"
 					(reference "USB_J1")
@@
 		(instances
 			(project "Main-Module"
+				(path "/acc63f22-7eb8-450a-9af4-da5f4b8157d9/066db7ca-fd8b-46d1-a06b-412eb11482f3"
+					(reference "#PWR037")
+					(unit 1)
+				)
+			)
+			(project "Main-Module"
 				(path "/c41b490b-5ab6-4438-aea0-388670bb08f4/b23d16a1-3c5b-4321-8b30-5d6992e2f62d"
 					(reference "#PWR037")
@@
 		(instances
 			(project "Main-Module"
+				(path "/acc63f22-7eb8-450a-9af4-da5f4b8157d9/066db7ca-fd8b-46d1-a06b-412eb11482f3"
+					(reference "#PWR039")
+					(unit 1)
+				)
+			)
+			(project "Main-Module"
 				(path "/c41b490b-5ab6-4438-aea0-388670bb08f4/b23d16a1-3c5b-4321-8b30-5d6992e2f62d"
 					(reference "#PWR039")
@@
 		(instances
 			(project "Main-Module"
+				(path "/acc63f22-7eb8-450a-9af4-da5f4b8157d9/066db7ca-fd8b-46d1-a06b-412eb11482f3"
+					(reference "#PWR036")
+					(unit 1)
+				)
+			)
+			(project "Main-Module"
 				(path "/c41b490b-5ab6-4438-aea0-388670bb08f4/b23d16a1-3c5b-4321-8b30-5d6992e2f62d"
 					(reference "#PWR036")
@@
 		(instances
 			(project "Main-Module"
+				(path "/acc63f22-7eb8-450a-9af4-da5f4b8157d9/066db7ca-fd8b-46d1-a06b-412eb11482f3"
+					(reference "USB_R2")
+					(unit 1)
+				)
+			)
+			(project "Main-Module"
 				(path "/c41b490b-5ab6-4438-aea0-388670bb08f4/b23d16a1-3c5b-4321-8b30-5d6992e2f62d"
 					(reference "USB_R2")
@@
 		)
 		(instances
+			(project "Main-Module"
+				(path "/acc63f22-7eb8-450a-9af4-da5f4b8157d9/066db7ca-fd8b-46d1-a06b-412eb11482f3"
+					(reference "USB_R1")
+					(unit 1)
+				)
+			)
 			(project "Main-Module"
 				(path "/c41b490b-5ab6-4438-aea0-388670bb08f4/b23d16a1-3c5b-4321-8b30-5d6992e2f62d"
@@
 			)
 		)
-		(property "Footprint" "ESDA7P60:ZDO_1610_STM"
+		(property "Footprint" "ESDA7P60_1U1M:ZDO_1610_STM"
 			(at 71.12 55.88 0)
 			(effects
@@
 		)
 		(instances
+			(project "Main-Module"
+				(path "/acc63f22-7eb8-450a-9af4-da5f4b8157d9/066db7ca-fd8b-46d1-a06b-412eb11482f3"
+					(reference "USB_CR1")
+					(unit 1)
+				)
+			)
 			(project "Main-Module"
 				(path "/c41b490b-5ab6-4438-aea0-388670bb08f4/b23d16a1-3c5b-4321-8b30-5d6992e2f62d"
@@
 		(instances
 			(project "Main-Module"
+				(path "/acc63f22-7eb8-450a-9af4-da5f4b8157d9/066db7ca-fd8b-46d1-a06b-412eb11482f3"
+					(reference "#PWR041")
+					(unit 1)
+				)
+			)
+			(project "Main-Module"
 				(path "/c41b490b-5ab6-4438-aea0-388670bb08f4/b23d16a1-3c5b-4321-8b30-5d6992e2f62d"
 					(reference "#PWR041")
@@
 		(instances
 			(project "Main-Module"
+				(path "/acc63f22-7eb8-450a-9af4-da5f4b8157d9/066db7ca-fd8b-46d1-a06b-412eb11482f3"
+					(reference "#PWR038")
+					(unit 1)
+				)
+			)
+			(project "Main-Module"
 				(path "/c41b490b-5ab6-4438-aea0-388670bb08f4/b23d16a1-3c5b-4321-8b30-5d6992e2f62d"
 					(reference "#PWR038")
@@
 		(instances
 			(project "Main-Module"
+				(path "/acc63f22-7eb8-450a-9af4-da5f4b8157d9/066db7ca-fd8b-46d1-a06b-412eb11482f3"
+					(reference "#PWR040")
+					(unit 1)
+				)
+			)
+			(project "Main-Module"
 				(path "/c41b490b-5ab6-4438-aea0-388670bb08f4/b23d16a1-3c5b-4321-8b30-5d6992e2f62d"
 					(reference "#PWR040")
@@
 		(instances
 			(project "Main-Module"
-				(path "/c41b490b-5ab6-4438-aea0-388670bb08f4/b23d16a1-3c5b-4321-8b30-5d6992e2f62d"
+				(path "/acc63f22-7eb8-450a-9af4-da5f4b8157d9/066db7ca-fd8b-46d1-a06b-412eb11482f3"
+					(reference "USB_TP1")
+					(unit 1)
+				)
+			)
+			(project "Main-Module"
+				(path "/c41b490b-5ab6-4438-aea0-388670bb08f4/b23d16a1-3c5b-4321-8b30-5d6992e2f62d"
