File: Common/Microcontroller.kicad_sch (KiCad schematic)
At the start: 14 parts

Commit message: Updating Schematics
Parts:
- renumbered MIC_C4 to MIC_C?, MIC_C2 to MIC_C?, MIC_C10 to MIC_C?, MIC_C7 to MIC_C?, MIC_C9 to MIC_C?, MIC_C6 to MIC_C?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
