File: Common/Microcontroller.kicad_sch (KiCad schematic)
At the start: 14 parts

Commit message: Made MC more generic
Connections:
- net accel_clk renamed SPI3_clk
- net accel_int1 renamed DIN_1
- net accel_int2 renamed DIN_2
- net accel_miso renamed SPI3_miso
- net accel_mosi renamed SPI3_mosi
- net flash_clk renamed SPI1_clk
- net flash_miso renamed SPI1_miso
- net flash_mosi renamed SPI1_mosi
- net pres_clk renamed SPI2_clk
- net pres_miso renamed SPI2_miso
- net pres_mosi renamed SPI2_mosi
