File: Main-Module/pcb/Main-Module.kicad_sch (KiCad schematic)
At the start: 22 parts, among them J1 Conn_02x10_Odd_Even, SW1 SW_DIP_x03, U1 W25Q128JVS, U2 MCP130-xxxxTT, U3 STM32H503RBTx

Commit message: Created microcontroller schematic
Parts:
- removed C10: 4.7uF, Capacitor_SMD:C_0603_1608Metric_Pad1.08x0.95mm_HandSolder, symbol Device:C
- removed C11, C3, C4, C5, C7, C9: 100nF, Capacitor_SMD:C_0603_1608Metric_Pad1.08x0.95mm_HandSolder, symbol Device:C
- removed C12: 1uF, Capacitor_SMD:C_0603_1608Metric_Pad1.08x0.95mm_HandSolder, symbol Device:C
- removed C6, C8: 2.2uF, Capacitor_SMD:C_0603_1608Metric_Pad1.08x0.95mm_HandSolder, symbol Device:C
- removed R1: 10k, Resistor_SMD:R_0603_1608Metric_Pad0.98x0.95mm_HandSolder, symbol Device:R_US
- removed SW1: SW_DIP_x03, Button_Switch_THT:SW_DIP_SPSTx03_Slide_9.78x9.8mm_W7.62mm_P2.54mm, symbol Switch:SW_DIP_x03
- removed U2: MCP130-xxxxTT, Package_TO_SOT_SMD:SOT-23, symbol Power_Supervisor:MCP130-xxxxTT
- removed U3: STM32H503RBTx, Package_QFP:LQFP-64_10x10mm_P0.5mm, symbol MCU_ST_STM32H5:STM32H503RBTx
Other:
- added sheet Microcontroller (Microcontroller.kicad_sch)
