File: Radio-Module/pcb/Flash.kicad_sch (KiCad schematic)
At the start: 3 parts, among them U1 W25Q128JVS

Commit message: Updating Schematics
Changed lines of the file:
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@@
 		)
 	)
-	(label "flash_mosi"
-		(at 147.32 100.33 0)
+	(hierarchical_label "flash_clk"
+		(shape input)
+		(at 147.32 97.79 180)
 		(fields_autoplaced yes)
 		(effects
@@
 				(size 1.27 1.27)
 			)
-			(justify left bottom)
-		)
-	)
-	(label "flash_clk"
-		(at 147.32 97.79 0)
+			(justify right)
+		)
+	)
+	(hierarchical_label "flash_mosi"
+		(shape input)
+		(at 147.32 100.33 180)
 		(fields_autoplaced yes)
 		(effects
@@
 				(size 1.27 1.27)
 			)
-			(justify left bottom)
-		)
-	)
-	(label "flash_miso"
-		(at 147.32 102.87 0)
+			(justify right)
+		)
+	)
+	(hierarchical_label "flash_miso"
+		(shape output)
+		(at 147.32 102.87 180)
 		(fields_autoplaced yes)
 		(effects
@@
 				(size 1.27 1.27)
 			)
-			(justify left bottom)
+			(justify right)
 		)
 	)
@@
 		(instances
 			(project ""
+				(path "/acc63f22-7eb8-450a-9af4-da5f4b8157d9/e039269b-c792-4448-9404-ba0f836b2ed0"
+					(reference "#PWR01")
+					(unit 1)
+				)
+			)
+			(project ""
 				(path "/e9d5c669-dec8-476e-8ce1-59a609c9ea65"
 					(reference "#PWR01")
@@
 		(instances
 			(project ""
+				(path "/acc63f22-7eb8-450a-9af4-da5f4b8157d9/e039269b-c792-4448-9404-ba0f836b2ed0"
+					(reference "#PWR02")
+					(unit 1)
+				)
+			)
+			(project ""
 				(path "/e9d5c669-dec8-476e-8ce1-59a609c9ea65"
 					(reference "#PWR02")
@@
 		(instances
 			(project ""
+				(path "/acc63f22-7eb8-450a-9af4-da5f4b8157d9/e039269b-c792-4448-9404-ba0f836b2ed0"
+					(reference "#PWR03")
+					(unit 1)
+				)
+			)
+			(project ""
 				(path "/e9d5c669-dec8-476e-8ce1-59a609c9ea65"
 					(reference "#PWR03")
@@
 		(instances
 			(project ""
+				(path "/acc63f22-7eb8-450a-9af4-da5f4b8157d9/e039269b-c792-4448-9404-ba0f836b2ed0"
+					(reference "C2")
+					(unit 1)
+				)
+			)
+			(project ""
 				(path "/e9d5c669-dec8-476e-8ce1-59a609c9ea65"
 					(reference "C2")
@@
 		)
 		(instances
+			(project ""
+				(path "/acc63f22-7eb8-450a-9af4-da5f4b8157d9/e039269b-c792-4448-9404-ba0f836b2ed0"
+					(reference "#PWR04")
+					(unit 1)
+				)
+			)
 			(project ""
 				(path "/e9d5c669-dec8-476e-8ce1-59a609c9ea65"
@@
 		(instances
 			(project ""
+				(path "/acc63f22-7eb8-450a-9af4-da5f4b8157d9/e039269b-c792-4448-9404-ba0f836b2ed0"
+					(reference "C1")
+					(unit 1)
+				)
+			)
+			(project ""
 				(path "/e9d5c669-dec8-476e-8ce1-59a609c9ea65"
 					(reference "C1")
@@
 		(instances
 			(project ""
-				(path "/e9d5c669-dec8-476e-8ce1-59a609c9ea65"
+				(path "/acc63f22-7eb8-450a-9af4-da5f4b8157d9/e039269b-c792-4448-9404-ba0f836b2ed0"
 					(reference "U1")
 					(unit 1)
 				)
 			)
-		)
-	)
-	(sheet_instances
-		(path "/"
-			(page "1")
-		)
-	)
+			(project ""
+				(path "/e9d5c669-dec8-476e-8ce1-59a609c9ea65"
+					(reference "U1")
+					(unit 1)
+				)
+			)
+		)
+	)
