File: Recovery-Module/pcb/Pyro-Controller.kicad_sch (KiCad schematic)
At the start: 0 parts

Commit message: Started Pyro Controller Sch.
Parts:
- added Q1: NMOS, symbol Simulation_SPICE:NMOS
- added R1, R2, R3, R4, R5: R_US, PYRO_R1, symbol Device:R_US
Connections:
- new net: R1.1, R2.2
- new net: Q1.1 (D), R3.1, R5.1
- new net: R3.2, R4.2
- new net: Q1.2 (G), R1.2
- new net GNDD: Q1.3 (S), R2.1, R4.1
