File: Pyro-Controller/pcb/Pyro-Controller/PyroController.kicad_sch (KiCad schematic)
At the start: 5 parts, among them U1 SI7232DN-T1-GE3

Commit message: Picked new (singular) nMOS for pyro controller. Finished board routing.
Parts:
- removed U1: SI7232DN-T1-GE3, footprints:SQJ500AEP-T1_GE3_VIS, symbol Si7232DN_T1_G3:SI7232DN-T1-GE3
- added Q1: SiS454DN, Package_SO:Vishay_PowerPAK_1212-8_Single, symbol Transistor_FET:SiS454DN
Connections:
- net GNDD: now also Q1.1 (S), Q1.2 (S), Q1.3 (S)
- net Output: now also Q1.5 (D)
- net at R2.2: now also Q1.4 (G)
Changed lines of the file:
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@@
+	(wire
+		(pts
+			(xy 115.57 77.47) (xy 162.56 77.47)
+		)
+		(stroke
+			(width 0)
+			(type default)
+		)
+	)
 	(wire
 		(pts
@@
 		(pts
 			(xy 172.72 77.47) (xy 172.72 81.28)
-		)
-		(stroke
-			(width 0)
-			(type default)
-		)
-	)
-	(wire
-		(pts
-			(xy 115.57 77.47) (xy 162.56 77.47)
 		)
 		(stroke
@@
 	)
 	(symbol
-		(lib_id "Si7232DN_T1_G3:SI7232DN-T1-GE3")
-		(at 107.95 87.63 0)
+		(lib_id "Transistor_FET:SiS454DN")
+		(at 113.03 87.63 0)
 		(unit 1)
 		(exclude_from_sim no)
@@
 		(on_board yes)
 		(dnp no)
-		(property "Reference" "U1"
-			(at 137.16 87.376 0)
-			(effects
-				(font
-					(size 1.524 1.524)
+		(fields_autoplaced yes)
+		(property "Reference" "Q1"
+			(at 119.38 86.3599 0)
+			(effects
+				(font
+					(size 1.27 1.27)
 				)
 				(justify left)
 			)
 		)
-		(property "Value" "SI7232DN-T1-GE3"
-			(at 137.16 85.0899 0)
-			(effects
-				(font
-					(size 1.524 1.524)
+		(property "Value" "SiS454DN"
+			(at 119.38 88.8999 0)
+			(effects
+				(font
+					(size 1.27 1.27)
 				)
 				(justify left)
 			)
 		)
-		(property "Footprint" "footprints:SQJ500AEP-T1_GE3_VIS"
-			(at 107.95 87.63 0)
+		(property "Footprint" "Package_SO:Vishay_PowerPAK_1212-8_Single"
+			(at 118.11 89.535 0)
 			(effects
 				(font
@@
 					(italic yes)
 				)
-				(hide yes)
-			)
-		)
-		(property "Datasheet" "SI7232DN-T1-GE3"
-			(at 107.95 87.63 0)
-			(effects
-				(font
-					(size 1.27 1.27)
-					(italic yes)
-				)
-				(hide yes)
-			)
-		)
-		(property "Description" ""
-			(at 107.95 87.63 0)
-			(effects
-				(font
-					(size 1.27 1.27)
-				)
-				(hide yes)
-			)
+				(justify left)
+				(hide yes)
+			)
+		)
+		(property "Datasheet" "https://www.vishay.com/docs/66707/sis454dn.pdf"
+			(at 118.11 91.44 0)
+			(effects
+				(font
+					(size 1.27 1.27)
+				)
+				(justify left)
+				(hide yes)
+			)
+		)
+		(property "Description" "35A Id, 20V Vds, N-Channel MOSFET, PowerPAK 1212-8 Single"
+			(at 113.03 87.63 0)
+			(effects
+				(font
+					(size 1.27 1.27)
+				)
+				(hide yes)
+			)
+		)
+		(pin "2"
+		)
+		(pin "1"
+		)
+		(pin "5"
 		)
 		(pin "4"
 		)
-		(pin "2"
-		)
 		(pin "3"
 		)
-		(pin "1"
-		)
 		(instances
-			(project "Pyro-Controller"
+			(project ""
 				(path "/3d6591d1-15d3-4f90-b463-ad4ce370627d/d3fae8d6-dc5c-4ad1-8056-ef8170011280"
-					(reference "U1")
+					(reference "Q1")
 					(unit 1)
 				)

Commit message: Added testpoint to Pyro Controller
Parts:
- added TP1, TP2, TP3: TestPoint, TestPoint:TestPoint_Loop_D2.54mm_Drill1.5mm_Beaded, symbol Connector:TestPoint
Connections:
- net GNDD: now also TP3.1
- net Input: now also TP1.1
- net Output: now also TP2.1
