File: IMU/pcb/Sensors.kicad_sch (KiCad schematic)
At the start: 5 parts, among them U6 MS5607-02BA, U7 ADXL375BCCZ

Commit message: Updated IMU schematic
Parts:
- removed U7: ADXL375BCCZ, Package_LGA:LGA-14_3x5mm_P0.8mm_LayoutBorder1x6y, symbol 2024-07-18_00-52-40:ADXL375BCCZ
- added U2: LSM6DSL, Package_LGA:LGA-14_3x2.5mm_P0.5mm_LayoutBorder3x4y, symbol Sensor_Motion:LSM6DSL
- renumbered C18 to C?, C20 to C?, C19 to C?, U6 to U?
Connections:
- net +3.3V: now also U2.5 (VDDIO), U2.8 (VDD)
- net GNDD: now also U2.12 (CS), U2.2 (SDX), U2.3 (SCX), U2.6 (GND), U2.7 (GND)
- new net imu_int1: U2.4 (INT1)
- new net imu_int2: U2.9 (INT2)
- new net imu_miso: U2.14 (SDA)
- new net imu_mosi: U2.1 (SDO/SA0)
- new net imu_sclk: U2.13 (SCL)
- no-connect marks 3 -> 0
