File: IMU/pcb/_autosave-_autosave-IMU.kicad_pcb (KiCad board)
At the start: 2 copper layers, 40.8 x 40.8 mm, 6 parts, among them J2 Conn_01x10_Socket, U1 MS5607-02BA, U2 LSM6DSL

Commit message: last semester changes
Routing:
- net GNDD: track 30.2 -> 89.1 mm, vias 0 -> 2
- net +3.3V: track 33.2 -> 46.2 mm, vias 0 -> 2
- net /sensors/imu_int2: track 21.4 -> 31.9 mm
Other:
- board outline removed
