File: IMU/pcb/IMU.kicad_sch (KiCad schematic)
At the start: 1 part, among them J1 Conn_01x10_Socket

Commit message: last semester changes
Parts:
- removed J1: Conn_01x10_Socket, symbol Connector:Conn_01x10_Socket
- added J2: Conn_01x10_Socket, Connector_PinHeader_2.54mm:PinHeader_1x10_P2.54mm_Vertical, symbol Connector:Conn_01x10_Socket
Connections:
- net +3.3V: now also J2.1 (Pin_1)
- net GNDD: now also J2.10 (Pin_10)
- net sensors/imu_int1: now also J2.2 (Pin_2)
- net sensors/imu_int2: now also J2.3 (Pin_3)
- net sensors/imu_miso: now also J2.5 (Pin_5)
- net sensors/imu_mosi: now also J2.4 (Pin_4)
- net sensors/imu_sclk: now also J2.6 (Pin_6)
- net sensors/pres_miso: now also J2.9 (Pin_9)
- net sensors/pres_mosi: now also J2.8 (Pin_8)
- net sensors/pres_sclk: now also J2.7 (Pin_7)
Changed lines of the file:
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@@
-	(wire
-		(pts
-			(xy 204.47 97.79) (xy 204.47 100.33)
-		)
-		(stroke
-			(width 0)
-			(type default)
-		)
-	)
 	(wire
 		(pts
@@
 	(wire
 		(pts
+			(xy 204.47 71.12) (xy 204.47 74.93)
+		)
+		(stroke
+			(width 0)
+			(type default)
+		)
+	)
+	(wire
+		(pts
+			(xy 204.47 74.93) (xy 207.01 74.93)
+		)
+		(stroke
+			(width 0)
+			(type default)
+		)
+	)
+	(wire
+		(pts
 			(xy 179.07 87.63) (xy 207.01 87.63)
 		)
@@
 	(wire
 		(pts
-			(xy 204.47 97.79) (xy 207.01 97.79)
+			(xy 207.01 97.79) (xy 205.74 97.79)
+		)
+		(stroke
+			(width 0)
+			(type default)
+		)
+	)
+	(wire
+		(pts
+			(xy 205.74 97.79) (xy 205.74 100.33)
 		)
 		(stroke
@@
 	(wire
 		(pts
-			(xy 200.66 74.93) (xy 207.01 74.93)
-		)
-		(stroke
-			(width 0)
-			(type default)
-		)
-	)
-	(wire
-		(pts
 			(xy 179.07 77.47) (xy 207.01 77.47)
 		)
@@
 			(width 0)
 			(type default)
+		)
+	)
+	(symbol
+		(lib_id "power:GNDD")
+		(at 205.74 100.33 0)
+		(unit 1)
+		(exclude_from_sim no)
+		(in_bom yes)
+		(on_board yes)
+		(dnp no)
+		(fields_autoplaced yes)
+		(property "Reference" "#PWR02"
+			(at 205.74 106.68 0)
+			(effects
+				(font
+					(size 1.27 1.27)
+				)
+				(hide yes)
+			)
+		)
+		(property "Value" "GNDD"
+			(at 205.74 104.14 0)
+			(effects
+				(font
+					(size 1.27 1.27)
+				)
+			)
+		)
+		(property "Footprint" ""
+			(at 205.74 100.33 0)
+			(effects
+				(font
+					(size 1.27 1.27)
+				)
+				(hide yes)
+			)
+		)
+		(property "Datasheet" ""
+			(at 205.74 100.33 0)
+			(effects
+				(font
+					(size 1.27 1.27)
+				)
+				(hide yes)
+			)
+		)
+		(property "Description" "Power symbol creates a global label with name \"GNDD\" , digital ground"
+			(at 205.74 100.33 0)
+			(effects
+				(font
+					(size 1.27 1.27)
+				)
+				(hide yes)
+			)
+		)
+		(pin "1"
+		)
+		(instances
+			(project ""
+				(path "/92f0fe4f-546b-4686-ae0e-a4b165f18304"
+					(reference "#PWR02")
+					(unit 1)
+				)
+			)
+		)
+	)
+	(symbol
+		(lib_id "power:+3.3V")
+		(at 204.47 71.12 0)
+		(unit 1)
+		(exclude_from_sim no)
+		(in_bom yes)
+		(on_board yes)
+		(dnp no)
+		(fields_autoplaced yes)
+		(property "Reference" "#PWR03"
+			(at 204.47 74.93 0)
+			(effects
+				(font
+					(size 1.27 1.27)
+				)
+				(hide yes)
+			)
+		)
+		(property "Value" "+3.3V"
+			(at 204.47 66.04 0)
+			(effects
+				(font
+					(size 1.27 1.27)
+				)
+			)
+		)
+		(property "Footprint" ""
+			(at 204.47 71.12 0)
+			(effects
+				(font
+					(size 1.27 1.27)
+				)
+				(hide yes)
+			)
+		)
+		(property "Datasheet" ""
+			(at 204.47 71.12 0)
+			(effects
+				(font
+					(size 1.27 1.27)
+				)
+				(hide yes)
+			)
+		)
+		(property "Description" "Power symbol creates a global label with name \"+3.3V\""
+			(at 204.47 71.12 0)
+			(effects
+				(font
+					(size 1.27 1.27)
+				)
+				(hide yes)
+			)
+		)
+		(pin "1"
+		)
+		(instances
+			(project ""
+				(path "/92f0fe4f-546b-4686-ae0e-a4b165f18304"
+					(reference "#PWR03")
+					(unit 1)
+				)
+			)
 		)
 	)
@@
 		(dnp no)
 		(fields_autoplaced yes)
-		(property "Reference" "J1"
+		(property "Reference" "J2"
 			(at 213.36 85.0899 0)
 			(effects
@@
 			)
 		)
-		(property "Footprint" ""
+		(property "Footprint" "Connector_PinHeader_2.54mm:PinHeader_1x10_P2.54mm_Vertical"
 			(at 212.09 85.09 0)
 			(effects
@@
 			)
 		)
+		(pin "10"
+		)
+		(pin "5"
+		)
+		(pin "1"
+		)
+		(pin "2"
+		)
+		(pin "4"
+		)
+		(pin "8"
+		)
+		(pin "7"
+		)
+		(pin "9"
+		)
 		(pin "3"
 		)
-		(pin "7"
-		)
-		(pin "9"
-		)
-		(pin "2"
-		)
-		(pin "5"
-		)
-		(pin "8"
-		)
 		(pin "6"
-		)
-		(pin "10"
-		)
-		(pin "1"
-		)
-		(pin "4"
 		)
 		(instances
 			(project ""
 				(path "/92f0fe4f-546b-4686-ae0e-a4b165f18304"
-					(reference "J1")
+					(reference "J2")
 					(unit 1)
 				)
-			)
-		)
-	)
-	(symbol
-		(lib_id "power:+3.3V")
-		(at 200.66 74.93 0)
-		(unit 1)
-		(exclude_from_sim no)
-		(in_bom yes)
-		(on_board yes)
-		(dnp no)
-		(fields_autoplaced yes)
-		(property "Reference" "#PWR02"
-			(at 200.66 78.74 0)
-			(effects
-				(font
-					(size 1.27 1.27)
-				)
-				(hide yes)
-			)
-		)
-		(property "Value" "+3.3V"
-			(at 200.66 69.85 0)
-			(effects
-				(font
-					(size 1.27 1.27)
-				)
-			)
-		)
-		(property "Footprint" ""
-			(at 200.66 74.93 0)
-			(effects
-				(font
-					(size 1.27 1.27)
-				)
-				(hide yes)
-			)
-		)
-		(property "Datasheet" ""
-			(at 200.66 74.93 0)
-			(effects
-				(font
-					(size 1.27 1.27)
-				)
-				(hide yes)
-			)
-		)
-		(property "Description" "Power symbol creates a global label with name \"+3.3V\""
-			(at 200.66 74.93 0)
-			(effects
-				(font
-					(size 1.27 1.27)
-				)
-				(hide yes)
-			)
-		)
-		(pin "1"
-		)
-		(instances
-			(project ""
-				(path "/92f0fe4f-546b-4686-ae0e-a4b165f18304"
-					(reference "#PWR02")
-					(unit 1)
-				)
-			)
-		)
-	)
-	(symbol
-		(lib_id "power:GNDD")
-		(at 204.47 100.33 0)
-		(unit 1)
-		(exclude_from_sim no)
-		(in_bom yes)
-		(on_board yes)
-		(dnp no)
-		(fields_autoplaced yes)
-		(property "Reference" "#PWR03"
-			(at 204.47 106.68 0)
-			(effects
-				(font
-					(size 1.27 1.27)
-				)
-				(hide yes)
-			)
-		)
-		(property "Value" "GNDD"
-			(at 204.47 104.14 0)
-			(effects
-				(font
-					(size 1.27 1.27)
-				)
-			)
-		)
-		(property "Footprint" ""
-			(at 204.47 100.33 0)
-			(effects
-				(font
-					(size 1.27 1.27)
-				)
-				(hide yes)
-			)
-		)
-		(property "Datasheet" ""
-			(at 204.47 100.33 0)
-			(effects
-				(font
-					(size 1.27 1.27)
-				)
-				(hide yes)
-			)
-		)
-		(property "Description" "Power symbol creates a global label with name \"GNDD\" , digital ground"
-			(at 204.47 100.33 0)
-			(effects
-				(font
-					(size 1.27 1.27)
-				)
-				(hide yes)
-			)
-		)
-		(pin "1"
-		)
-		(instances
-			(project ""
-				(path "/92f0fe4f-546b-4686-ae0e-a4b165f18304"
-					(reference "#PWR03")
-					(unit 1)
-				)

Commit message: Finished IMU Rev 1
Parts:
- removed J2: Conn_01x10_Socket, Connector_PinHeader_2.54mm:PinHeader_1x10_P2.54mm_Vertical, symbol Connector:Conn_01x10_Socket
- added FID1, FID2, FID3: Fiducial, Fiducial:Fiducial_1mm_Mask2mm, symbol Mechanical:Fiducial
- added J1, J2: Conn_01x06_Pin, Connector_PinHeader_2.54mm:PinHeader_1x06_P2.54mm_Vertical, symbol Connector:Conn_01x06_Pin
Connections:
- net +3.3V: now also J1.1 (Pin_1), J2.1 (Pin_1)
- net GNDD: now also J1.6 (Pin_6), J2.6 (Pin_6)
- net sensors/imu_int1: now also J1.5 (Pin_5)
- net sensors/imu_int2: now also J2.5 (Pin_5)
- net sensors/imu_miso: now also J1.2 (Pin_2)
- net sensors/imu_mosi: now also J1.3 (Pin_3)
- net sensors/imu_sclk: now also J1.4 (Pin_4)
- net sensors/pres_miso: now also J2.2 (Pin_2)
- net sensors/pres_mosi: now also J2.3 (Pin_3)
- net sensors/pres_sclk: now also J2.4 (Pin_4)

Commit message: IMU test board rev 2
Parts:
- removed J1, J2: Conn_01x06_Pin, Connector_PinHeader_2.54mm:PinHeader_1x06_P2.54mm_Vertical, symbol Connector:Conn_01x06_Pin
- added J1, J2: Conn_01x07_Pin, Connector_PinHeader_2.54mm:PinHeader_1x07_P2.54mm_Vertical, symbol Connector:Conn_01x07_Pin
Connections:
- net +3.3V: now also J1.1 (Pin_1), J2.1 (Pin_1)
- net GNDD: now also J1.7 (Pin_7), J2.7 (Pin_7)
- net sensors/imu_int1: now also J1.5 (Pin_5)
- net sensors/imu_int2: now also J2.5 (Pin_5)
- net sensors/imu_miso: now also J1.2 (Pin_2)
- net sensors/imu_mosi: now also J1.3 (Pin_3)
- net sensors/imu_sclk: now also J1.4 (Pin_4)
- net sensors/pres_miso: now also J2.2 (Pin_2)
- net sensors/pres_mosi: now also J2.3 (Pin_3)
- net sensors/pres_sclk: now also J2.4 (Pin_4)
- new net sensors/imu_cs: J1.6 (Pin_6)
- new net sensors/pres_cs: J2.6 (Pin_6)
Other:
- sheet sensors ports: added imu_cs, pres_cs; removed none
