File: IMU/pcb/IMU.kicad_pcb (KiCad board)
At the start: 2 copper layers, 22.9 x 22.9 mm, 11 parts, among them J1 Conn_01x06_Pin, J2 Conn_01x06_Pin, U1 MS5607-02BA, U2 LSM6DSL

Commit message: IMU test board rev 2
Parts:
- J1, J2: value Conn_01x06_Pin -> Conn_01x07_Pin; footprint Connector_PinHeader_2.54mm:PinHeader_1x06_P2.54mm_Vertical -> Connector_PinHeader_2.54mm:PinHeader_1x07_P2.54mm_Vertical; moved to B.Cu
- moved C3 0.37 mm to (134.0, 99.0)
- moved J1 0.29 mm to (141.7, 91.3), turned to 180 degrees
- turned J2 to 180 degrees
Connections:
- J1 pad 6: GNDD -> /sensors/imu_cs
- J2 pad 6: GNDD -> /sensors/pres_cs
- U1 pad 4: GNDD -> /sensors/pres_cs
- U1 pad 5: GNDD -> /sensors/pres_cs
- U2 pad 12: GNDD -> /sensors/imu_cs
Routing:
- net /sensors/pres_cs: track 0.00 -> 15.9 mm, vias 0 -> 1
- net /sensors/imu_cs: track 0.00 -> 12.1 mm
- net GNDD: track 15.6 -> 11.3 mm, vias 11 -> 8
Other:
- board text added: "IMU Rev. 2"
- board text removed: "IMU Rev. 1"

Commit message: Syncing up!
Parts:
- C2: footprint Capacitor_Tantalum_SMD:CP_EIA-3216-18_Kemet-A_Pad1.58x1.35mm_HandSolder -> Capacitor_SMD:C_0603_1608Metric_Pad1.08x0.95mm_HandSolder
- moved C2 0.75 mm to (130.1, 101.1)
Connections:
- U2 pad 1: /sensors/imu_mosi -> /sensors/imu_miso
- U2 pad 14: /sensors/imu_miso -> /sensors/imu_mosi
Routing:
- net +3.3V: track 4.66 -> 0.09 mm
- net /sensors/imu_mosi: track 13.1 -> 15.0 mm
- net /sensors/imu_miso: track 17.4 -> 15.7 mm
- net GNDD: track 11.3 -> 10.6 mm
Changed lines of the file:
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@@
 			(psa4output no)
 			(plot_black_and_white yes)
-			(plotinvisibletext no)
 			(sketchpadsonfab no)
 			(plotpadnumbers no)
@@
 		(embedded_fonts no)
 	)
-	(footprint "Capacitor_Tantalum_SMD:CP_EIA-3216-18_Kemet-A_Pad1.58x1.35mm_HandSolder"
+	(footprint "Capacitor_SMD:C_0603_1608Metric_Pad1.08x0.95mm_HandSolder"
 		(layer "F.Cu")
-		(at 129.3125 101.092 -90)
-		(descr "Tantalum Capacitor SMD Kemet-A (3216-18 Metric), IPC_7351 nominal, (Body size from: http://www.kemet.com/Lists/ProductCatalog/Attachments/253/KEM_TC101_STD.pdf), generated with kicad-footprint-generator")
-		(tags "capacitor tantalum")
+		(at 130.058 101.0975 -90)
+		(descr "Capacitor SMD 0603 (1608 Metric), square (rectangular) end terminal, IPC-7351 nominal with elongated pad for handsoldering. (Body size source: IPC-SM-782 page 76, https://www.pcb-3d.com/wordpress/wp-content/uploads/ipc-sm-782a_amendment_1_and_2.pdf), generated with kicad-footprint-generator")
+		(tags "capacitor handsolder")
 		(property "Reference" "C2"
-			(at 0 1.7945 90)
+			(at 0 1.5405 270)
 			(layer "F.SilkS")
 			(effects
@@
 		)
 		(property "Value" "10uF"
-			(at 0 1.75 90)
+			(at 0 1.43 270)
 			(layer "F.Fab")
 			(effects
@@
 		(property "Datasheet" "https://content.kemet.com/datasheets/KEM_T2005_T491.pdf"
 			(at 0 0 270)
-			(unlocked yes)
 			(layer "F.Fab")
 			(hide yes)
@@
 		(property "Description" "Unpolarized capacitor"
 			(at 0 0 270)
-			(unlocked yes)
 			(layer "F.Fab")
 			(hide yes)
@@
 		(attr smd)
 		(fp_line
-			(start -2.485 0.935)
-			(end 1.6 0.935)
-			(stroke
-				(width 0.12)
-				(type solid)
-			)
-			(layer "F.SilkS")
-		)
-		(fp_line
-			(start -2.485 -0.935)
-			(end -2.485 0.935)
+			(start -0.146267 0.51)
+			(end 0.146267 0.51)
 			(stroke
 				(width 0.12)
@@
 		)
 		(fp_line
-			(start 1.6 -0.935)
-			(end -2.485 -0.935)
+			(start -0.146267 -0.51)
+			(end 0.146267 -0.51)
 			(stroke
 				(width 0.12)
@@
 		)
 		(fp_line
-			(start -2.48 1.05)
-			(end -2.48 -1.05)
+			(start -1.65 0.73)
+			(end -1.65 -0.73)
 			(stroke
 				(width 0.05)
@@
 		)
 		(fp_line
-			(start 2.48 1.05)
-			(end -2.48 1.05)
+			(start 1.65 0.73)
+			(end -1.65 0.73)
 			(stroke
 				(width 0.05)
@@
 		)
 		(fp_line
-			(start -2.48 -1.05)
-			(end 2.48 -1.05)
+			(start -1.65 -0.73)
+			(end 1.65 -0.73)
 			(stroke
 				(width 0.05)
@@
 		)
 		(fp_line
-			(start 2.48 -1.05)
-			(end 2.48 1.05)
+			(start 1.65 -0.73)
+			(end 1.65 0.73)
 			(stroke
 				(width 0.05)
@@
 		)
 		(fp_line
-			(start -1.6 0.8)
-			(end 1.6 0.8)
-			(stroke
-				(width 0.1)
-				(type solid)
-			)
-			(layer "F.Fab")
-		)
-		(fp_line
-			(start 1.6 0.8)
-			(end 1.6 -0.8)
+			(start -0.8 0.4)
+			(end -0.8 -0.4)
 			(stroke
 				(width 0.1)
@@
 		)
 		(fp_line
-			(start -1.6 -0.4)
-			(end -1.6 0.8)
+			(start 0.8 0.4)
+			(end -0.8 0.4)
 			(stroke
 				(width 0.1)
@@
 		)
 		(fp_line
-			(start -1.2 -0.8)
-			(end -1.6 -0.4)
+			(start -0.8 -0.4)
+			(end 0.8 -0.4)
 			(stroke
 				(width 0.1)
@@
 		)
 		(fp_line
-			(start 1.6 -0.8)
-			(end -1.2 -0.8)
+			(start 0.8 -0.4)
+			(end 0.8 0.4)
 			(stroke
 				(width 0.1)
@@
 		)
 		(fp_text user "${REFERENCE}"
-			(at 0 1.75 90)
+			(at 0 0 270)
 			(layer "F.Fab")
 			(effects
 				(font
-					(size 0.8 0.8)
-					(thickness 0.12)
+					(size 0.4 0.4)
+					(thickness 0.06)
 				)
 			)
 		)
 		(pad "1" smd roundrect
-			(at -1.4375 0 270)
-			(size 1.575 1.35)
+			(at -0.8625 0 270)
+			(size 1.075 0.95)
 			(layers "F.Cu" "F.Mask" "F.Paste")
-			(roundrect_rratio 0.185185)
+			(roundrect_rratio 0.25)
 			(net 1 "+3.3V")
 			(pintype "passive")
 		)
 		(pad "2" smd roundrect
-			(at 1.4375 0 270)
-			(size 1.575 1.35)
+			(at 0.8625 0 270)
+			(size 1.075 0.95)
 			(layers "F.Cu" "F.Mask" "F.Paste")
-			(roundrect_rratio 0.185185)
+			(roundrect_rratio 0.25)
 			(net 2 "GNDD")
 			(pintype "passive")
 		)
 		(embedded_fonts no)
-		(model "${KICAD8_3DMODEL_DIR}/Capacitor_Tantalum_SMD.3dshapes/CP_EIA-3216-18_Kemet-A.wrl"
+		(model "${KICAD9_3DMODEL_DIR}/Capacitor_SMD.3dshapes/C_0603_1608Metric.wrl"
 			(offset
 				(xyz 0 0 0)
@@
 			(layers "F.Cu" "F.Mask" "F.Paste")
 			(roundrect_rratio 0.25)
-			(net 9 "/sensors/imu_mosi")
+			(net 6 "/sensors/imu_miso")
 			(pinfunction "SDO/SA0")
 			(pintype "bidirectional")
@@
 			(layers "F.Cu" "F.Mask" "F.Paste")
 			(roundrect_rratio 0.25)
-			(net 6 "/sensors/imu_miso")
+			(net 9 "/sensors/imu_mosi")
 			(pinfunction "SDA")
 			(pintype "bidirectional")
@@
 	)
 	(segment
-		(start 131.452 100.0565)
-		(end 131.05 99.6545)
-		(width 0.3556)
-		(layer "F.Cu")
-		(net 1)
-	)
-	(segment
-		(start 131.452 100.596)
-		(end 131.452 100.0565)
-		(width 0.3556)
-		(layer "F.Cu")
-		(net 1)
-	)
-	(segment
-		(start 133.1145 100.4335)
-		(end 133.1145 98.7135)
-		(width 0.3556)
+		(start 134.408 101.198)
+		(end 134.392 101.214)
+		(width 0.2)
 		(layer "F.Cu")
-		(net 1)
+		(net 2)
 	)
 	(segment
-		(start 131.05 99.6545)
-		(end 129.3125 99.6545)
+		(start 130.058 102.0215)
+		(end 130.058 103.23)
 		(width 0.3556)
 		(layer "F.Cu")
-		(net 1)
+		(net 2)
 	)
 	(segment
@@
 	)
 	(segment
-		(start 135.038 101.214)
-		(end 133.777 101.214)
-		(width 0.2)
-		(layer "F.Cu")
-		(net 2)
-	)
-	(segment
 		(start 132.1145 99.576)
 		(end 132.1065 99.568)
@@
 	)
 	(segment
-		(start 129.3125 102.5295)
-		(end 129.3125 104.14)
-		(width 0.3556)
+		(start 134.884 101.198)
+		(end 134.408 101.198)
+		(width 0.2)
 		(layer "F.Cu")
 		(net 2)
@@
 	)
 	(segment
+		(start 134.392 101.214)
+		(end 133.777 101.214)
+		(width 0.2)
+		(layer "F.Cu")
+		(net 2)
+	)
+	(segment
 		(start 134.8575 98.3035)
 		(end 135.265 97.896)
@@
 		(net 2)
 	)
-	(segment
-		(start 135.138 101.314)
-		(end 135.038 101.214)
-		(width 0.2)
-		(layer "F.Cu")
-		(net 2)
-	)
 	(via
-		(at 129.3125 104.14)
+		(at 130.058 103.23)
 		(size 0.6)
 		(drill 0.3)
@@
 	)
 	(via
-		(at 135.138 101.314)
+		(at 134.884 101.198)
 		(size 0.6)
 		(drill 0.3)
@@
 	)
 	(segment
-		(start 133.3765 103.251)
-		(end 134.1385 103.251)
-		(width 0.2)
-		(layer "F.Cu")
-		(net 6)
-	)
-	(segment
-		(start 137.17 93.578)
-		(end 141.752 93.578)
+		(start 133.777 102.214)
+		(end 134.544203 102.214)
 		(width 0.2)
 		(layer "F.Cu")
@@
 	)
 	(segment
-		(start 133.1145 102.2585)
-		(end 133.1145 102.989)
+		(start 134.544203 102.214)
+		(end 134.884 101.874203)
 		(width 0.2)
 		(layer "F.Cu")
@@
 	)
 	(segment
-		(start 133.1145 102.989)
-		(end 133.3765 103.251)
+		(start 137.17 93.578)
+		(end 141.752 93.578)
 		(width 0.2)
 		(layer "F.Cu")
@@
 	)
 	(via
-		(at 134.1385 103.251)
+		(at 134.884 101.874203)
 		(size 0.6)
 		(drill 0.3)
@@
 	)
 	(segment
-		(start 137.17 93.578)
+		(start 134.1385 96.6095)
+		(end 137.17 93.578)
+		(width 0.2)
+		(layer "B.Cu")
+		(net 6)
+	)
+	(segment
+		(start 134.1385 101.128703)
 		(end 134.1385 96.6095)
 		(width 0.2)
@@
 	)
 	(segment
-		(start 134.1385 96.6095)
-		(end 134.1385 103.251)
+		(start 134.884 101.874203)
+		(end 134.1385 101.128703)
 		(width 0.2)
 		(layer "B.Cu")
@@
 	)
 	(segment
-		(start 137.0565 102.214)
-		(end 137.17 102.214)
+		(start 136.154 103.23)
+		(end 133.3555 103.23)
 		(width 0.2)
 		(layer "F.Cu")
@@
 	)
 	(segment
-		(start 133.777 102.214)
-		(end 137.0565 102.214)
+		(start 133.1145 102.2585)
+		(end 133.1145 102.989)
+		(width 0.2)
+		(layer "F.Cu")
+		(net 9)
+	)
+	(segment
+		(start 133.3555 103.23)
+		(end 133.1145 102.989)
 		(width 0.2)
 		(layer "F.Cu")
@@
 	)
 	(via
-		(at 137.17 102.214)
+		(at 136.154 103.23)
 		(size 0.6)
 		(drill 0.3)
@@
 	)
 	(segment
-		(start 138.821 96.118)
-		(end 137.1865 97.7525)
+		(start 136.154 103.23)
+		(end 137.1865 102.1975)
 		(width 0.2)
 		(layer "B.Cu")
@@
 	(segment
 		(start 137.1865 97.7525)
-		(end 137.1865 102.214)
+		(end 138.821 96.118)
+		(width 0.2)
+		(layer "B.Cu")
+		(net 9)
+	)
+	(segment
+		(start 137.1865 102.1975)
+		(end 137.1865 97.7525)
 		(width 0.2)
 		(layer "B.Cu")
