File: Valve-Controller/pcb/Valve-Controller/Valve-Controller.kicad_sch (KiCad schematic)
At the start: 5 parts, among them J1 Screw_Terminal_01x02, J2 Conn_01x03_Socket

Commit message: Valve controller diode
Connections:
- net +3.3V renamed +12V

Commit message: Resized pin socket pitch to 2.54mm
Parts:
- J2: footprint Connector_PinSocket_2.00mm:PinSocket_1x03_P2.00mm_Vertical -> Connector_PinSocket_2.54mm:PinSocket_1x03_P2.54mm_Vertical
Changed lines of the file:
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@@
 			)
 		)
-		(property "Footprint" "Connector_PinSocket_2.00mm:PinSocket_1x03_P2.00mm_Vertical"
+		(property "Footprint" "Connector_PinSocket_2.54mm:PinSocket_1x03_P2.54mm_Vertical"
 			(at 99.06 77.47 0)
 			(effects

Commit message: Revert "Resolved recovery dev merge"
This reverts commit 81c4bbda93894cf9b120906f02d3dbab6bbd1e60, reversing
changes made to 220360569fc6c62025a0e7a68270d7f77f4a1f37.
Parts:
- J2: footprint Connector_PinSocket_2.54mm:PinSocket_1x03_P2.54mm_Vertical -> Connector_PinSocket_2.00mm:PinSocket_1x03_P2.00mm_Vertical
Changed lines of the file:
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@@
 			)
 		)
-		(property "Footprint" "Connector_PinSocket_2.54mm:PinSocket_1x03_P2.54mm_Vertical"
+		(property "Footprint" "Connector_PinSocket_2.00mm:PinSocket_1x03_P2.00mm_Vertical"
 			(at 99.06 77.47 0)
 			(effects
