File: Common/rowan-rocketry.kicad_blocks/USB-C PD Controller.kicad_block/USB-C PD Controller.kicad_sch (KiCad schematic)
At the start: 33 parts, among them J201 USB_C_Receptacle_USB2.0_16P, Q201 IRF9358, Q202 2N7002, Q203 BSL308PE, U201 USBLC6-2SC6, U202 CYPD3177-24LQ

Commit message: KiCAD schematic blocks are a thing now
Parts:
- renumbered D201 to D1, R212 to R3, R201 to R?, R208 to R?, R210 to R?, R207 to R?, U202 to U?, J201 to USB_J?, TP203 to USB_TP?, TP202 to USB_TP?, TP201 to USB_TP?, TP204 to USB_TP?, U201 to USB_U?
Connections:
- net DC_OUT: now also Q201.7 (D1), Q201.8 (D1); no longer Q201.5 (D2), Q201.6 (D2)
- net SAFE_5V_OUT: now also Q203.6 (D1); no longer Q203.4 (D2)
- net at D1.1 (K), Q201.1 (S1), R3.1: now also Q201.1 (S1); no longer Q201.3 (S2)
- net at C202.2, C203.2, D1.2 (A)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: now also Q201.2 (G1); no longer Q201.4 (G2)
- net at Q203.5 (S1): now also Q203.5 (S1); no longer Q203.2 (S2)
- net at Q203.1 (G1), R209.1, R213.2: now also Q203.1 (G1); no longer Q203.3 (G2)
