File: Ride-Along-Module/pcb/3v7 LiPo to 3v3 Supply.kicad_sch (KiCad schematic)
At the start: 5 parts

Commit message: More reuse blocks. Added battery circuit to ride along board
Parts:
- BT1: footprint Battery:BatteryHolder_MPD_BH-18650-PC2 -> Connector_JST:JST_PH_B2B-PH-K_1x02_P2.00mm_Vertical
- gave numbers to parts that had none: 4
Other:
- moved on the sheet: BT1, C17, C19, C20, U5

Commit message: Ride-Along Module Rev. 1
Parts:
- added D3: LED, LED_SMD:LED_0603_1608Metric, symbol Device:LED
- added R6: 1k, Resistor_SMD:R_0603_1608Metric, symbol Device:R_US
- added TP2, TP3, TP4: TestPoint, TestPoint:TestPoint_Loop_D2.60mm_Drill1.6mm_Beaded, symbol Connector:TestPoint
- BT1: value Battery_Cell -> LiPo Connector
- C16: renamed from C17; footprint Capacitor_SMD:C_0603_1608Metric_Pad1.08x0.95mm_HandSolder -> Capacitor_SMD:C_0603_1608Metric
- C17: renamed from C19; footprint Capacitor_SMD:C_0603_1608Metric_Pad1.08x0.95mm_HandSolder -> Capacitor_SMD:C_0603_1608Metric
- C18: renamed from C20; footprint Capacitor_SMD:C_0603_1608Metric_Pad1.08x0.95mm_HandSolder -> Capacitor_SMD:C_0603_1608Metric
- U3: renamed from U5; Purchase (none) -> https://www.digikey.com/en/products/detail/microchip-techno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
Connections:
- net +3.3V: now also R6.1, TP3.1
- net GNDD: now also D3.1 (K), TP2.1
- net V_BAT: now reaches BT1.1 (+), C16.1, U3.1 (VIN), U3.3 (ON/~{OFF})
- net V_BAT: now also TP4.1
- new net: D3.2 (A), R6.2
Other:
- company: (none) -> Rowan Rocketry
- title: (none) -> Ride-Along Module
- moved on the sheet: BT1
