File: Ride-Along-Module/pcb/USB-C Port.kicad_sch (KiCad schematic)
At the start: 6 parts, among them J1 USB_C_Receptacle_USB2.0_16P, U1 USBLC6-2SC6

Commit message: Ride-Along Module Rev. 1
Parts:
- D2: renamed from D1; Purchase (none) -> https://www.digikey.com/en/products/detail/rohm-semiconduct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
- J1: Purchase (none) -> https://www.digikey.com/en/products/detail/gct/USB4105-GF-A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
- R2: renamed from R1; footprint Resistor_SMD:R_0603_1608Metric_Pad0.98x0.95mm_HandSolder -> Resistor_SMD:R_0603_1608Metric
- R3: renamed from R2; footprint Resistor_SMD:R_0603_1608Metric_Pad0.98x0.95mm_HandSolder -> Resistor_SMD:R_0603_1608Metric
- U1: Purchase (none) -> https://www.digikey.com/en/products/detail/stmicroelectroni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
Other:
- company: (none) -> Rowan Rocketry
- title: (none) -> Ride-Along Module
Changed lines of the file:
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@@
 	(generator_version "9.0")
 	(paper "A4")
-	(text_box "Keep ESD protection circuitry (U1_usb, CR1_usb) as close to the connector as possible."
+	(title_block
+		(title "Ride-Along Module")
+		(date "2025-04-10")
+		(rev "1")
+		(company "Rowan Rocketry")
+	)
+	(text_box "Keep ESD protection circuitry (U1, D2) as close to the connector as possible."
 		(exclude_from_sim no)
 		(at 85.09 83.82 0)
@@
 		(stroke
 			(width 0)
-			(type default)
+			(type solid)
 		)
 		(fill
@@
 	(no_connect
 		(at 62.23 92.71)
-	)
-	(bus_entry
-		(at 95.25 40.64)
-		(size 2.54 2.54)
-		(stroke
-			(width 0)
-			(type default)
-		)
 	)
 	(wire
@@
 		)
 		(property "Description" "Very low capacitance ESD protection diode, 2 data-line, SOT-23-6"
+			(at 78.74 77.47 0)
+			(effects
+				(font
+					(size 1.27 1.27)
+				)
+				(hide yes)
+			)
+		)
+		(property "Purchase" "https://www.digikey.com/en/products/detail/stmicroelectronics/USBLC6-2SC6/1040559"
 			(at 78.74 77.47 0)
 			(effects
@@
 			)
 		)
+		(property "Purchase" "https://www.digikey.com/en/products/detail/gct/USB4105-GF-A/11198441"
+			(at 46.99 77.47 0)
+			(effects
+				(font
+					(size 1.27 1.27)
+				)
+				(hide yes)
+			)
+		)
 		(pin "B12"
 		)
@@
 		(dnp no)
 		(fields_autoplaced yes)
-		(property "Reference" "#PWR02"
+		(property "Reference" "#PWR07"
 			(at 46.99 106.68 0)
 			(effects
@@
 			(project "Radio-Module"
 				(path "/ba7b4294-8d75-4b9e-892f-fb52727887ec/b41619a2-11a0-4fcf-9c2d-b1ec93f6b99c"
-					(reference "#PWR02")
+					(reference "#PWR07")
 					(unit 1)
 				)
@@
 		(dnp no)
 		(fields_autoplaced yes)
-		(property "Reference" "#PWR03"
+		(property "Reference" "#PWR08"
 			(at 85.09 62.23 0)
 			(effects
@@
 			(project "Radio-Module"
 				(path "/ba7b4294-8d75-4b9e-892f-fb52727887ec/b41619a2-11a0-4fcf-9c2d-b1ec93f6b99c"
-					(reference "#PWR03")
+					(reference "#PWR08")
 					(unit 1)
 				)
@@
 		(dnp no)
 		(fields_autoplaced yes)
-		(property "Reference" "#PWR01"
+		(property "Reference" "#PWR06"
 			(at 39.37 106.68 0)
 			(effects
@@
 			(project "Radio-Module"
 				(path "/ba7b4294-8d75-4b9e-892f-fb52727887ec/b41619a2-11a0-4fcf-9c2d-b1ec93f6b99c"
-					(reference "#PWR01")
+					(reference "#PWR06")
 					(unit 1)
 				)
@@
 		(dnp no)
 		(fields_autoplaced yes)
-		(property "Reference" "D1"
+		(property "Reference" "D2"
 			(at 74.93 55.88 0)
 			(effects
@@
 		)
 		(property "Description" "Zener diode"
+			(at 74.93 62.23 0)
+			(effects
+				(font
+					(size 1.27 1.27)
+				)
+				(hide yes)
+			)
+		)
+		(property "Purchase" "https://www.digikey.com/en/products/detail/rohm-semiconductor/VS5V0UA1LAMTR/7902291?s=N4IgTCBcDaIGoGUCscAMBVAggRgDKYFkAVAJRAF0BfIA"
 			(at 74.93 62.23 0)
 			(effects
@@
 			(project ""
 				(path "/ba7b4294-8d75-4b9e-892f-fb52727887ec/b41619a2-11a0-4fcf-9c2d-b1ec93f6b99c"
-					(reference "D1")
+					(reference "D2")
 					(unit 1)
 				)
@@
 		(on_board yes)
 		(dnp no)
-		(property "Reference" "R2"
+		(property "Reference" "R3"
 			(at 107.95 70.358 90)
 			(effects
@@
 			)
 		)
-		(property "Footprint" "Resistor_SMD:R_0603_1608Metric_Pad0.98x0.95mm_HandSolder"
+		(property "Footprint" "Resistor_SMD:R_0603_1608Metric"
 			(at 108.204 73.914 90)
 			(effects
@@
 			(project "Radio-Module"
 				(path "/ba7b4294-8d75-4b9e-892f-fb52727887ec/b41619a2-11a0-4fcf-9c2d-b1ec93f6b99c"
-					(reference "R2")
+					(reference "R3")
 					(unit 1)
 				)
@@
 		(on_board yes)
 		(dnp no)
-		(property "Reference" "R1"
+		(property "Reference" "R2"
 			(at 107.95 62.484 90)
 			(effects
@@
 			)
 		)
-		(property "Footprint" "Resistor_SMD:R_0603_1608Metric_Pad0.98x0.95mm_HandSolder"
+		(property "Footprint" "Resistor_SMD:R_0603_1608Metric"
 			(at 108.204 66.294 90)
 			(effects
@@
 			(project "Radio-Module"
 				(path "/ba7b4294-8d75-4b9e-892f-fb52727887ec/b41619a2-11a0-4fcf-9c2d-b1ec93f6b99c"
-					(reference "R1")
+					(reference "R2")
 					(unit 1)
 				)
@@
 		(dnp no)
 		(fields_autoplaced yes)
-		(property "Reference" "#PWR06"
+		(property "Reference" "#PWR011"
 			(at 120.65 74.93 0)
 			(effects
@@
 			(project "Radio-Module"
 				(path "/ba7b4294-8d75-4b9e-892f-fb52727887ec/b41619a2-11a0-4fcf-9c2d-b1ec93f6b99c"
-					(reference "#PWR06")
+					(reference "#PWR011")
 					(unit 1)
 				)
@@
 		(dnp no)
 		(fields_autoplaced yes)
-		(property "Reference" "#PWR04"
+		(property "Reference" "#PWR09"
 			(at 78.74 91.44 0)
 			(effects
@@
 			(project "Radio-Module"
 				(path "/ba7b4294-8d75-4b9e-892f-fb52727887ec/b41619a2-11a0-4fcf-9c2d-b1ec93f6b99c"
-					(reference "#PWR04")
+					(reference "#PWR09")
 					(unit 1)
 				)
@@
 		(dnp no)
 		(fields_autoplaced yes)
-		(property "Reference" "#PWR05"
+		(property "Reference" "#PWR010"
 			(at 120.65 67.31 0)
 			(effects
@@
 			(project "Radio-Module"
 				(path "/ba7b4294-8d75-4b9e-892f-fb52727887ec/b41619a2-11a0-4fcf-9c2d-b1ec93f6b99c"
-					(reference "#PWR05")
-					(unit 1)
-				)
+					(reference "#PWR010")
+					(unit 1)
+				)
