File: Common/rowan-rocketry.kicad_blocks/IMU Sensors.kicad_block/IMU Sensors.kicad_sch (KiCad schematic)
At the start: 5 parts, among them U3 MS5607-02BA, U4 LSM6DSL

Commit message: More reuse blocks. Added battery circuit to ride along board
Parts:
- renumbered C14 to C?, C16 to C?, C15 to C?, U3 to U?, U4 to U?
Other:
- moved on the sheet: C?, U?

Commit message: Pos file for IMU rev 2
Connections:
- net GNDD: no longer U?.12 (CS), U?.4 (CSB), U?.5 (CSB)
- new net imu_cs: U?.12 (CS)
- new net pres_cs: U?.4 (CSB), U?.5 (CSB)
Other:
- moved on the sheet: C?, U?
